File: ai03-pcb-guide.kicad_sch (KiCad schematic)
At the start: 0 parts

Commit message: finished schematic
Parts:
- added C1: 1uF, Capacitor_SMD:C_0805_2012Metric, symbol Device:C_Small_US
- added C2, C3, C4, C5: 0.1uF, Capacitor_SMD:C_0805_2012Metric, symbol Device:C_Small_US
- added C6, C7: 22pF, Capacitor_SMD:C_0805_2012Metric, symbol Device:C_Small_US
- added D1, D2, D3, D4: D_Small, Diode_SMD:D_SOD-123, symbol Device:D_Small
- added F1: 500mA, Fuse:Fuse_1206_3216Metric, symbol Device:Polyfuse_Small
- added R1, R4: 10k, Fuse:Fuse_0805_2012Metric, symbol Device:R_Small_US
- added R2, R3: 22, Fuse:Fuse_0805_2012Metric, symbol Device:R_Small_US
- added SW1: SW_Push, random-keyboard-parts:SKQG-1155865, symbol Switch:SW_Push
- added SW2, SW3, SW4, SW5: SW_Push, MX_Alps_Hybrid:MX-Alps-Hybrid-1U, symbol Switch:SW_Push
- added U1: ATmega32U4-A, Package_QFP:TQFP-44_10x10mm_P0.8mm, symbol MCU_Microchip_ATmega:ATmega32U4-A
- added USB1: Molex-0548190589, random-keyboard-parts:Molex-0548190589, symbol random-keyboard-parts:Molex-0548190589
- added Y1: 16MHz, Crystal:Crystal_SMD_3225-4Pin_3.2x2.5mm, symbol Device:Crystal_GND24_Small
Connections:
- new net: R4.1, SW1.2, U1.13 (~{RESET})
- new net: C7.1, U1.16 (XTAL2), Y1.3
- new net: C6.2, U1.17 (XTAL1), Y1.1
- new net: R3.2, U1.3 (D-)
- new net: R1.1, U1.33 (~{HWB}/PE2)
- new net: R2.2, U1.4 (D+)
- new net: C1.1, U1.6 (UCAP)
- new net: D4.2 (A), SW5.1
- new net: D3.2 (A), SW4.1
- new net: D1.2 (A), SW2.1
- new net: D2.2 (A), SW3.1
- new net +5V: C2.1, C3.1, C4.1, C5.1, F1.2, R4.2, U1.14 (VCC), U1.2 (UVCC), U1.24 (AVCC), U1.34 (VCC), U1.44 (AVCC), U1.7 (VBUS)
- new net COL0: SW2.2, SW4.2, U1.29 (PB5)
- new net COL1: SW3.2, SW5.2, U1.28 (PB4)
- new net D+: R2.1, USB1.3 (D+)
- new net D-: R3.1, USB1.4 (D-)
- new net GND: C1.2, C2.2, C3.2, C4.2, C5.2, C6.1, C7.2, R1.2, SW1.1, U1.15 (GND), U1.23 (GND), U1.35 (GND), U1.43 (GND), U1.5 (UGND), USB1.1 (GND), USB1.6 (SHIELD), Y1.2, Y1.4
- new net ROW0: D1.1 (K), D2.1 (K), U1.27 (PD7)
- new net ROW1: D3.1 (K), D4.1 (K), U1.30 (PB6)
- new net VCC: F1.1, USB1.5 (VBUS)
- no-connect marks 0 -> 23
